Commit message: add left/right wrist cam

File: assets/embodiments/g1-omnipicker/agibot_g1_with_omnipicker.urdf (robot description, URDF)
Before this commit: robot agibot_g1_with_omni-picker, 54 links, 53 joints
Links:
- added link left_camera
- added link right_camera
Joints:
- added joint left_wrist_camera_joint: type fixed, parent left_camera_stand, child left_camera, origin xyz=0 -0.07754 0.028618 rpy=0 -1.117 1.5708
- added joint right_wrist_camera_joint: type fixed, parent right_camera_stand, child right_camera, origin xyz=0 -0.07754 0.028618 rpy=0 -1.117 1.5708
